File: 2623162-CarlosIgnacioMercado-Microarduino.kicad_sch (KiCad schematic)
At the start: 14 parts, among them J1 USB_A_UCC, J2 Header, U1 ATtiny85-20S

Commit message: cambios en el proyecto
Parts:
- D4: footprint Diode_SMD:D_MELF_Handsoldering -> Diode_SMD:D_MiniMELF
Changed lines of the file:
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@@
 			)
 		)
-		(property "Footprint" "Diode_SMD:D_MELF_Handsoldering"
+		(property "Footprint" "Diode_SMD:D_MiniMELF"
 			(at 43.18 72.39 0)
 			(effects
